File: main-board/main-board.kicad_pcb (KiCad board)
At the start: 4 copper layers, 170.8 x 119.4 mm, 203 parts, among them IC10 SN74AXC4T774RSVR, IC13 TPS2121RUXR, IC15 SN74AXC4T774RSVR, IC16 SN74AXC4T774RSVR, IC2 SN74AXC4T774RSVR, IC3 SN74AXC4T774RSVR, IC4 SN74AXC4T774RSVR, J1 Conn_01x08, J12 Conn_01x01_Socket, J2 Conn_01x08, J20 Conn_01x01_Pin, J37 Conn_01x03, J4 Conn_01x08, J47 Barrel Jack, J5 Conn_01x08, J66 Conn_01x01_Socket, J68 Conn_02x02_Odd_Even, J70 Conn_01x07, J71 Conn_02x01, J72 Conn_01x07, J73 Conn_01x03, J74 Conn_Boaxial, J8 Conn_01x16, P2 USB Micro, SW1 SW_SPDT, SW2 SW_SPDT, SW3 SW_SPDT, SW5 SW_Push, U1 FT4232HL, U11 TS5A23159DGS, U12 TS5A23159DGS, U13 TS5A23159DGS, U14 TS5A23159DGS, U17 74AHC244, U2 W25Q128JWSIQ, U24 TCA9554ADBQR, U25 TCA9554ADBQR, U27 SI5351A-B-GTR, U28 TS5A23159DGS, U3 TLV75801PDBV, U31 74AHC244, U9 74AHCT1G08, X2 OK322532.768KJBA4SL, Y1 Crystal_GND24, Y2 NX3225GA-25.000M-STD-CRG-2

Commit message: Before re-organizing the main board
Parts:
- removed the C97 at (39.5, 34.9)
- removed J1: Conn_01x08, Connector_PinSocket_2.54mm:PinSocket_1x06_P2.54mm_Vertical
- removed J2, J4, J5: Conn_01x08, Connector_PinSocket_2.54mm:PinSocket_1x09_P2.54mm_Vertical
- removed the J20 at (39.9, 31.3)
- removed J70, J72: Conn_01x07, Connector_PinSocket_2.54mm:PinSocket_1x07_P2.54mm_Vertical
- removed J8: Conn_01x16, Connector_PinSocket_2.54mm:PinSocket_1x16_P2.54mm_Vertical
- removed the U25 at (41.5, 25.6)
- J10, J3, J6, J7, J9: renamed from REF**; value PinHeader_2x16_P1.27mm_Vertical -> Conn_02x16_Odd_Even; footprint Connector_PinHeader_1.27mm:PinHeader_2x16_P1.27mm_Vertical -> Connector_PinHeader_1.27mm:PinHeader_2x16_P1.27mm_Horizontal
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Connections:
- C11 pad 1: +3.3V -> 3V3
- C12 pad 1: +3.3V -> 3V3
- C13 pad 1: +3.3V -> 3V3
- C15 pad 1: +3.3V -> 3V3
- C16 pad 1: /V_IO -> /VDD_IO
- C20 pad 1: /Vpm -> /5V
- C22 pad 1: /3V3_LDO -> 3V3
- C31 pad 1: +3.3V -> 3V3
- C32 pad 1: +3.3V -> 3V3
- C33 pad 1: +3.3V -> 3V3
- C34 pad 1: +3.3V -> 3V3
- C35 pad 1: /V_IO -> /VDD_IO
- C36 pad 1: /V_IO -> /VDD_IO
- C37 pad 1: /V_IO -> /VDD_IO
- C38 pad 1: /V_IO -> /VDD_IO
- C45 pad 1: +3.3V -> 3V3
- C46 pad 1: +3.3V -> 3V3
- C47 pad 1: +3.3V -> 3V3
- C48 pad 1: +3.3V -> 3V3
- C49 pad 1: /V_IO -> /VDD_IO
- C50 pad 1: +3.3V -> 3V3
- C60 pad 1: /Vpm -> /5V
- C61 pad 1: /Vpm -> /5V
- C63 pad 1: +3.3V -> 3V3
- C64 pad 1: +3.3V -> 3V3
- C66 pad 1: +3.3V -> 3V3
- C81 pad 1: +3.3V -> 3V3
- C82 pad 1: +3.3V -> 3V3
- C83 pad 2: +3.3V -> 3V3
- C85 pad 1: /V_IO -> /VDD_IO
- C86 pad 1: /V_IO -> /VDD_IO
- C89 pad 2: +3.3V -> 3V3
- C90 pad 1: /V_IO -> /VDD_IO
- C97 pad 1: +3.3V -> 3V3
- CG1 pad 12: /SDA -> /5V
- CG1 pad 13: /SCL -> /5V
- CG1 pad 6: unconnected-(CG1-TP_2-Pad6) -> /SCL
- CG1 pad 7: unconnected-(CG1-TP_3-Pad7) -> /SDA
- CG10 pad 12: /SDA -> /5V
- CG10 pad 13: /SCL -> /5V
- CG10 pad 6: unconnected-(CG10-TP_2-Pad6) -> /SCL
- CG10 pad 7: unconnected-(CG10-TP_3-Pad7) -> /SDA
- CG11 pad 12: /SDA -> /5V
- CG11 pad 13: /SCL -> /5V
- CG11 pad 6: unconnected-(CG11-TP_2-Pad6) -> /SCL
- CG11 pad 7: unconnected-(CG11-TP_3-Pad7) -> /SDA
- CG12 pad 12: /SDA -> /5V
- CG12 pad 13: /SCL -> /5V
- CG12 pad 20: /chewing-gums/Vout_8_diff -> /chewing-gums/Vout_12_diff
- CG12 pad 6: unconnected-(CG12-TP_2-Pad6) -> /SCL
- CG12 pad 7: unconnected-(CG12-TP_3-Pad7) -> /SDA
- CG2 pad 12: /SDA -> /5V
- CG2 pad 13: /SCL -> /5V
- CG2 pad 6: unconnected-(CG2-TP_2-Pad6) -> /SCL
- CG2 pad 7: unconnected-(CG2-TP_3-Pad7) -> /SDA
- CG3 pad 12: /SDA -> /5V
- CG3 pad 13: /SCL -> /5V
- CG3 pad 6: unconnected-(CG3-TP_2-Pad6) -> /SCL
- CG3 pad 7: unconnected-(CG3-TP_3-Pad7) -> /SDA
- CG4 pad 12: /SDA -> /5V
- CG4 pad 13: /SCL -> /5V
- CG4 pad 6: unconnected-(CG4-TP_2-Pad6) -> /SCL
- CG4 pad 7: unconnected-(CG4-TP_3-Pad7) -> /SDA
- CG5 pad 1: /chewing-gums/Vout_5_A -> /VDD_IO
- CG5 pad 12: /SDA -> /5V
- CG5 pad 13: /SCL -> /5V
- CG5 pad 2: /chewing-gums/Vout_5_A -> /VDD_IO
- CG5 pad 21: /chewing-gums/Vout_5_A -> /VDD_IO
- CG5 pad 6: unconnected-(CG5-TP_2-Pad6) -> /SCL
- CG5 pad 7: unconnected-(CG5-TP_3-Pad7) -> /SDA
- CG6 pad 12: /SDA -> /5V
- CG6 pad 13: /SCL -> /5V
- CG6 pad 6: unconnected-(CG6-TP_2-Pad6) -> /SCL
- CG6 pad 7: unconnected-(CG6-TP_3-Pad7) -> /SDA
- CG7 pad 12: /SDA -> /5V
- CG7 pad 13: /SCL -> /5V
- CG7 pad 6: unconnected-(CG7-TP_2-Pad6) -> /SCL
- CG7 pad 7: unconnected-(CG7-TP_3-Pad7) -> /SDA
- CG8 pad 12: /SDA -> /5V
- CG8 pad 13: /SCL -> /5V
- CG8 pad 6: unconnected-(CG8-TP_2-Pad6) -> /SCL
- CG8 pad 7: unconnected-(CG8-TP_3-Pad7) -> /SDA
- CG9 pad 12: /SDA -> /5V
- CG9 pad 13: /SCL -> /5V
- CG9 pad 6: unconnected-(CG9-TP_2-Pad6) -> /SCL
- CG9 pad 7: unconnected-(CG9-TP_3-Pad7) -> /SDA
- D7 pad 2: /3V3_LDO -> 3V3
- IC10 pad 13: /V_IO -> /VDD_IO
- IC10 pad 14: +3.3V -> 3V3
- IC10 pad 15: +3.3V -> 3V3
- IC10 pad 16: +3.3V -> 3V3
- IC13 pad 1: /Vpm -> /5V
- IC13 pad 8: /Vpm -> /5V
- IC15 pad 13: /V_IO -> /VDD_IO
- IC15 pad 14: +3.3V -> 3V3
- IC16 pad 13: /V_IO -> /VDD_IO
- IC16 pad 14: +3.3V -> 3V3
- IC2 pad 13: /V_IO -> /VDD_IO
- IC2 pad 14: +3.3V -> 3V3
- IC2 pad 15: +3.3V -> 3V3
- IC2 pad 16: +3.3V -> 3V3
- IC2 pad 5: +3.3V -> 3V3
- IC3 pad 13: /V_IO -> /VDD_IO
- IC3 pad 14: +3.3V -> 3V3
- IC3 pad 15: +3.3V -> 3V3
- IC3 pad 16: +3.3V -> 3V3
- IC3 pad 5: +3.3V -> 3V3
- IC4 pad 13: /V_IO -> /VDD_IO
- IC4 pad 14: +3.3V -> 3V3
- IC4 pad 15: +3.3V -> 3V3
- IC4 pad 16: +3.3V -> 3V3
- IC4 pad 5: +3.3V -> 3V3
- J10 pad 1: (no net) -> /REF
- J10 pad 10: (no net) -> /SCL
- J10 pad 11: (no net) -> GND
- J10 pad 12: (no net) -> GND
- J10 pad 13: (no net) -> 3V3
- J10 pad 14: (no net) -> 3V3
- J10 pad 15: (no net) -> GND
- J10 pad 16: (no net) -> GND
- J10 pad 17: (no net) -> /5V
- J10 pad 18: (no net) -> /5V
- J10 pad 19: (no net) -> GND
- J10 pad 2: (no net) -> /REF
- J10 pad 20: (no net) -> GND
- J10 pad 21: (no net) -> unconnected-(J10-Pin_21-Pad21)
- J10 pad 22: (no net) -> unconnected-(J10-Pin_22-Pad22)
- J10 pad 23: (no net) -> unconnected-(J10-Pin_23-Pad23)
- J10 pad 24: (no net) -> unconnected-(J10-Pin_24-Pad24)
- J10 pad 25: (no net) -> unconnected-(J10-Pin_25-Pad25)
- J10 pad 26: (no net) -> unconnected-(J10-Pin_26-Pad26)
- J10 pad 27: (no net) -> unconnected-(J10-Pin_27-Pad27)
- J10 pad 28: (no net) -> unconnected-(J10-Pin_28-Pad28)
- J10 pad 29: (no net) -> unconnected-(J10-Pin_29-Pad29)
- J10 pad 3: (no net) -> GND
- J10 pad 30: (no net) -> unconnected-(J10-Pin_30-Pad30)
- J10 pad 31: (no net) -> unconnected-(J10-Pin_31-Pad31)
- J10 pad 32: (no net) -> unconnected-(J10-Pin_32-Pad32)
- J10 pad 4: (no net) -> GND
- J10 pad 5: (no net) -> /A3V3
- J10 pad 6: (no net) -> /A3V3
- J10 pad 7: (no net) -> GND
- J10 pad 8: (no net) -> GND
- J10 pad 9: (no net) -> /SDA
- J3 pad 1: (no net) -> GND
- J3 pad 10: (no net) -> /chewing-gums/GPIO_11
- J3 pad 11: (no net) -> /chewing-gums/GPIO_12
- J3 pad 12: (no net) -> /chewing-gums/GPIO_13
- J3 pad 13: (no net) -> /chewing-gums/GPIO_14
- J3 pad 14: (no net) -> /chewing-gums/GPIO_15
- J3 pad 15: (no net) -> /chewing-gums/GPIO_16
- J3 pad 16: (no net) -> /chewing-gums/GPIO_17
- J3 pad 17: (no net) -> GND
- J3 pad 18: (no net) -> GND
- J3 pad 19: (no net) -> /chewing-gums/GPIO_18
- J3 pad 2: (no net) -> GND
- J3 pad 20: (no net) -> /chewing-gums/GPIO_19
- J3 pad 21: (no net) -> /chewing-gums/GPIO_20
- J3 pad 22: (no net) -> /chewing-gums/GPIO_21
- J3 pad 23: (no net) -> /chewing-gums/GPIO_22
- J3 pad 24: (no net) -> /chewing-gums/GPIO_22
- J3 pad 25: (no net) -> /chewing-gums/GPIO_24
- J3 pad 26: (no net) -> /chewing-gums/GPIO_25
- J3 pad 27: (no net) -> GND
- J3 pad 28: (no net) -> GND
- J3 pad 29: (no net) -> unconnected-(J3-Pin_29-Pad29)
- J3 pad 3: (no net) -> /chewing-gums/Vout_3_diff
- J3 pad 30: (no net) -> unconnected-(J3-Pin_30-Pad30)
- J3 pad 31: (no net) -> unconnected-(J3-Pin_31-Pad31)
- J3 pad 32: (no net) -> unconnected-(J3-Pin_32-Pad32)
- J3 pad 4: (no net) -> /chewing-gums/Vout_3_B
- J3 pad 5: (no net) -> /chewing-gums/Vout_3_A
- J3 pad 6: (no net) -> /chewing-gums/Vout_3_A
- J3 pad 7: (no net) -> GND
- J3 pad 8: (no net) -> GND
- J3 pad 9: (no net) -> /chewing-gums/GPIO_10
- J6 pad 1: (no net) -> /chewing-gums/Vout_4_diff
- J6 pad 10: (no net) -> /chewing-gums/EXIT_VALUE
- J6 pad 11: (no net) -> /chewing-gums/BOOT_SEL
- J6 pad 12: (no net) -> unconnected-(J6-Pin_12-Pad12)
- J6 pad 13: (no net) -> GND
- J6 pad 14: (no net) -> GND
- J6 pad 15: (no net) -> /chewing-gums/GPIO_2
- J6 pad 16: (no net) -> /chewing-gums/GPIO_3
- J6 pad 17: (no net) -> /chewing-gums/GPIO_4
- J6 pad 18: (no net) -> /chewing-gums/GPIO_5
- J6 pad 19: (no net) -> /chewing-gums/GPIO_6
- J6 pad 2: (no net) -> /chewing-gums/Vout_4_B
- J6 pad 20: (no net) -> /chewing-gums/GPIO_7
- J6 pad 21: (no net) -> /chewing-gums/GPIO_8
- J6 pad 22: (no net) -> /chewing-gums/GPIO_9
- J6 pad 23: (no net) -> GND
- J6 pad 24: (no net) -> GND
- J6 pad 25: (no net) -> /chewing-gums/SPI_FLASH_CS0
- J6 pad 26: (no net) -> /chewing-gums/SPI_FLASH_CS1
- J6 pad 27: (no net) -> /chewing-gums/SPI_FLASH_SD2
- J6 pad 28: (no net) -> /chewing-gums/SPI_FLASH_SD3
- J6 pad 29: (no net) -> /chewing-gums/SPI_FLASH_SD0
- J6 pad 3: (no net) -> /chewing-gums/Vout_4_A
- J6 pad 30: (no net) -> /chewing-gums/SPI_FLASH_SD1
- J6 pad 31: (no net) -> /chewing-gums/SPI_FLASH_SCK
- J6 pad 32: (no net) -> unconnected-(J6-Pin_32-Pad32)
- J6 pad 4: (no net) -> /chewing-gums/Vout_4_A
- J6 pad 5: (no net) -> GND
- J6 pad 6: (no net) -> GND
- J6 pad 7: (no net) -> /chewing-gums/nRST
- J6 pad 8: (no net) -> /chewing-gums/EXEC_FLASH
- J6 pad 9: (no net) -> /chewing-gums/EXIT_VALID
- J68 pad 1: +3.3V -> 3V3
- J68 pad 3: +3.3V -> 3V3
- J7 pad 1: (no net) -> /chewing-gums/Vout_6_diff
- J7 pad 10: (no net) -> /chewing-gums/SPI_S_SCK
- J7 pad 11: (no net) -> /chewing-gums/SPI_S_MOSI
- J7 pad 12: (no net) -> /chewing-gums/SPI_S_MISO
- J7 pad 13: (no net) -> GND
- J7 pad 14: (no net) -> GND
- J7 pad 15: (no net) -> /chewing-gums/JTAG_TCK
- J7 pad 16: (no net) -> /chewing-gums/JTAG_TMS
- J7 pad 17: (no net) -> /chewing-gums/JTAG_TD0
- J7 pad 18: (no net) -> /chewing-gums/JTAG_TDI
- J7 pad 19: (no net) -> GND
- J7 pad 2: (no net) -> /chewing-gums/Vout_6_B
- J7 pad 20: (no net) -> GND
- J7 pad 21: (no net) -> /chewing-gums/UART_TX
- J7 pad 22: (no net) -> /chewing-gums/UART_RX
- J7 pad 23: (no net) -> GND
- J7 pad 24: (no net) -> GND
- J7 pad 25: (no net) -> /chewing-gums/Vout_5_diff
- J7 pad 26: (no net) -> /chewing-gums/Vout_5_B
- J7 pad 27: (no net) -> /VDD_IO
- J7 pad 28: (no net) -> /VDD_IO
- J7 pad 29: (no net) -> GND
- J7 pad 3: (no net) -> /chewing-gums/Vout_6_A
- J7 pad 30: (no net) -> GND
- J7 pad 31: (no net) -> /chewing-gums/clk
- J7 pad 32: (no net) -> GND
- J7 pad 4: (no net) -> /chewing-gums/Vout_6_A
- J7 pad 5: (no net) -> GND
- J7 pad 6: (no net) -> GND
- J7 pad 7: (no net) -> /chewing-gums/GPIO_0
- J7 pad 8: (no net) -> /chewing-gums/GPIO_1
- J7 pad 9: (no net) -> /chewing-gums/SPI_S_CS
- J71 pad 1: +3.3V -> 3V3
- J9 pad 1: (no net) -> GND
- J9 pad 10: (no net) -> /chewing-gums/Vout_11_A
- J9 pad 11: (no net) -> GND
- J9 pad 12: (no net) -> GND
- J9 pad 13: (no net) -> /chewing-gums/Vout_10_diff
- J9 pad 14: (no net) -> /chewing-gums/Vout_10_B
- J9 pad 15: (no net) -> /chewing-gums/Vout_10_A
- J9 pad 16: (no net) -> /chewing-gums/Vout_10_A
- J9 pad 17: (no net) -> /chewing-gums/Vout_9_diff
- J9 pad 18: (no net) -> /chewing-gums/Vout_9_B
- J9 pad 19: (no net) -> /chewing-gums/Vout_9_A
- J9 pad 2: (no net) -> GND
- J9 pad 20: (no net) -> /chewing-gums/Vout_9_A
- J9 pad 21: (no net) -> GND
- J9 pad 22: (no net) -> GND
- J9 pad 23: (no net) -> /chewing-gums/Vout_8_diff
- J9 pad 24: (no net) -> /chewing-gums/Vout_8_B
- J9 pad 25: (no net) -> /chewing-gums/Vout_8_A
- J9 pad 26: (no net) -> /chewing-gums/Vout_8_A
- J9 pad 27: (no net) -> /chewing-gums/Vout_7_diff
- J9 pad 28: (no net) -> /chewing-gums/Vout_7_B
- J9 pad 29: (no net) -> /chewing-gums/Vout_7_A
- J9 pad 3: (no net) -> /chewing-gums/Vout_12_diff
- J9 pad 30: (no net) -> /chewing-gums/Vout_7_A
- J9 pad 31: (no net) -> GND
- J9 pad 32: (no net) -> GND
- J9 pad 4: (no net) -> /chewing-gums/Vout_12_B
- J9 pad 5: (no net) -> /chewing-gums/Vout_12_A
- J9 pad 6: (no net) -> /chewing-gums/Vout_12_A
- J9 pad 7: (no net) -> /chewing-gums/Vout_11_diff
- J9 pad 8: (no net) -> /chewing-gums/Vout_11_B
- J9 pad 9: (no net) -> /chewing-gums/Vout_11_A
- L1 pad 1: +3.3V -> 3V3
- L2 pad 1: +3.3V -> 3V3
- R103 pad 2: +3.3V -> 3V3
- R108 pad 1: +3.3V -> 3V3
- R109 pad 1: +3.3V -> 3V3
- R110 pad 1: +3.3V -> 3V3
- R111 pad 1: +3.3V -> 3V3
- R14 pad 2: /V_IO -> /VDD_IO
- R24 pad 1: +3.3V -> 3V3
- R25 pad 1: +3.3V -> 3V3
- R26 pad 1: +3.3V -> 3V3
- R27 pad 1: /V_IO -> /VDD_IO
- R45 pad 2: /Vpm -> /5V
- R46 pad 2: /3V3_LDO -> 3V3
- R6 pad 1: /V_IO -> /VDD_IO
- R7 pad 1: /V_IO -> /VDD_IO
- R78 pad 2: /V_IO -> /VDD_IO
- R8 pad 1: /V_IO -> /VDD_IO
- R84 pad 1: +3.3V -> 3V3
- R9 pad 1: /V_IO -> /VDD_IO
- SW1 pad 1: /V_IO -> /VDD_IO
- SW2 pad 1: /V_IO -> /VDD_IO
- SW3 pad 1: /V_IO -> /VDD_IO
- U1 pad 20: +3.3V -> 3V3
- U1 pad 31: +3.3V -> 3V3
- U1 pad 42: +3.3V -> 3V3
- U1 pad 50: +3.3V -> 3V3
- U1 pad 56: +3.3V -> 3V3
- U11 pad 8: +3.3V -> 3V3
- U12 pad 8: +3.3V -> 3V3
- U13 pad 8: +3.3V -> 3V3
- U14 pad 8: +3.3V -> 3V3
- U17 pad 20: +3.3V -> 3V3
- U2 pad 8: /V_IO -> /VDD_IO
- U24 pad 1: +3.3V -> 3V3
- U24 pad 16: +3.3V -> 3V3
- U25 pad 16: +3.3V -> 3V3
- U27 pad 1: +3.3V -> 3V3
- U27 pad 7: /V_IO -> /VDD_IO
- U28 pad 8: +3.3V -> 3V3
- U3 pad 1: /Vpm -> /5V
- U3 pad 5: /3V3_LDO -> 3V3
- U31 pad 20: +3.3V -> 3V3
- U4 pad 3: /3V3 -> 3V3
- U4 pad 4: /3V3 -> 3V3
- U9 pad 1: +3.3V -> 3V3
- U9 pad 5: +3.3V -> 3V3
- X2 pad 4: /V_IO -> /VDD_IO
Routing:
- net 3V3: track 0.00 -> 347.2 mm, vias 0 -> 16
- net /VDD_IO: track 0.00 -> 220.7 mm, vias 0 -> 4
- net /chewing-gums/EN_12: track 0.00 -> 202.8 mm
- net /chewing-gums/EN_11: track 0.00 -> 189.8 mm
- net /chewing-gums/EN_10: track 0.00 -> 176.2 mm
- net /chewing-gums/EN_9: track 0.00 -> 162.7 mm
- net /chewing-gums/EN_8: track 0.00 -> 149.2 mm
- net /chewing-gums/EN_7: track 0.00 -> 135.9 mm
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- added copper zone on B.Cu, net /5V
- added copper zone on F.Cu, net /5V
- added copper zone on F.Cu, net /VUSB
- added copper zone on B.Cu, net 3V3
- added copper zone on F.Cu, net 3V3
- added copper zone on F.Cu, net GND
- added copper zone on F.Cu, net Net-(U1-OSCI)
- added copper zone on F.Cu, net Net-(U1-OSCO)
Other:
- board size 170.8 x 119.4 mm -> 170.8 x 120.2 mm
- board text added: "3V3"
- board text added: "5V"
- board text added: "USB & FTDI"
- board text added: "VDDio"
- board text removed: "5V regulator"
- board text removed: "FTDI"
- board text removed: "GPIO mux"
- board text removed: "Have one power per layer using the two central layers"
- board text removed: "LEDs"
- board text removed: "UART & JTAG LS"
- board text removed: "USB"

Commit message: tested main board side by side
Parts:
- removed D12, D13, D14, D15, D16, D17, D18, D19, D20, D21, D22, D23, D24, D25, D26, D27: LED, LED_SMD:LED_0603_1608Metric
- removed R100, R112, R113, R114, R115, R116, R48, R66, R67, R68, R69, R80, R81, R97, R98, R99: 1k, Resistor_SMD:R_0603_1608Metric
- removed U17, U31: 74AHC244, Package_SO:TSSOP-20_4.4x6.5mm_P0.65mm
- moved C32 186.7 mm to (-69.8, 86.1)
- moved C46 186.7 mm to (-81.5, 78.8)
- moved C64 186.7 mm to (-81.3, 67.2)
- moved IC15 186.7 mm to (-85.6, 65.6)
- moved R110 186.7 mm to (-90.3, 77.6)
- moved U12 186.7 mm to (-92.8, 95.0)
- moved C11 186.7 mm to (-82.6, 54.2)
- moved C16 186.7 mm to (-81.0, 83.9)
- moved C33 186.7 mm to (-81.8, 80.8)
- moved C34 186.7 mm to (-87.7, 77.6)
- moved C35 186.7 mm to (-81.8, 82.4)
- moved C36 186.7 mm to (-86.1, 77.6)
- moved C45 186.7 mm to (-80.6, 92.6)
- moved C47 186.7 mm to (-87.7, 92.6)
- moved C48 186.7 mm to (-94.1, 89.5)
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Routing:
- net /REF: track 386.8 -> 208.2 mm
- net /A3V3: track 346.1 -> 173.7 mm
- net /chewing-gums/Vout_3_A: track 143.9 -> 12.3 mm
- net /SCL: track 318.9 -> 190.4 mm
- net 3V3: track 347.2 -> 221.4 mm
- net /chewing-gums/Vout_3_B: track 128.2 -> 5.14 mm
- net /chewing-gums/Vout_3_diff: track 175.0 -> 54.1 mm
- net /VDD_IO: track 220.7 -> 103.5 mm
- net /chewing-gums/Vout_6_A: track 128.6 -> 11.7 mm
- net /chewing-gums/Vout_4_A: track 126.7 -> 12.2 mm
- net /chewing-gums/EN_6: track 113.2 -> 0.00 mm
- net /chewing-gums/EN_7: track 135.9 -> 25.0 mm
- net /chewing-gums/EN_8: track 149.2 -> 38.8 mm
- net /chewing-gums/EN_9: track 162.7 -> 53.2 mm
- net /chewing-gums/EN_10: track 176.2 -> 67.5 mm
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Other:
- board text added: "Programmer & LS"
- board text removed: "BOOT sgn"
- board text removed: "CLK"
- board text removed: "Custom power sources (or other things)"
- board text removed: "GPIOs"
- board text removed: "JTAG"
- board text removed: "PWR"
- board text removed: "SPI S"
- board text removed: "SPI flash"
- board text removed: "UART"
- board text removed: "VDDio"

Commit message: Before re-routing programmer
Parts:
- removed C97: 0.1u, Capacitor_SMD:C_0603_1608Metric
- removed J10, J6, J7, J9: Conn_02x16_Odd_Even, Connector_PinHeader_1.27mm:PinHeader_2x16_P1.27mm_Horizontal
- removed J20: Conn_01x01_Pin, Connector_PinHeader_2.54mm:PinHeader_1x01_P2.54mm_Vertical
- removed U25: TCA9554ADBQR, Package_SO:SSOP-16_3.9x4.9mm_P0.635mm
- added C14: 0.1u, Capacitor_SMD:C_0603_1608Metric, F.Cu at (156.1, 57.5)
- added C21: 0.1u, Capacitor_SMD:C_0603_1608Metric, F.Cu at (114.7, 142.7)
- added J2: Conn_02x16_Odd_Even, Connector_PinHeader_1.27mm:PinHeader_2x16_P1.27mm_Horizontal, F.Cu at (127.7, 152.7)
- added J3: Conn_02x16_Odd_Even, Connector_PinHeader_1.27mm:PinHeader_2x16_P1.27mm_Horizontal, F.Cu at (150.4, 152.5)
- added J4: Conn_02x16_Odd_Even, Connector_PinHeader_1.27mm:PinHeader_2x16_P1.27mm_Horizontal, F.Cu at (172.9, 152.5)
- added J5: Conn_02x16_Odd_Even, Connector_PinHeader_1.27mm:PinHeader_2x16_P1.27mm_Horizontal, F.Cu at (196.1, 152.5)
- added U5: ~, heep_footprints:adc-dac, F.Cu at (175.5, 59.7)
- added U6: ~, Package_DFN_QFN:WQFN-24-1EP_4x4mm_P0.5mm_EP2.6x2.6mm, F.Cu at (159.5, 59.6)
- added U7: ~, Package_DFN_QFN:WQFN-24-1EP_4x4mm_P0.5mm_EP2.6x2.6mm, F.Cu at (112.1, 146.6)
- J37: footprint Connector_PinSocket_2.54mm:PinSocket_1x03_P2.54mm_Vertical -> Connector_PinSocket_2.54mm:PinSocket_1x03_P2.54mm_Vertical_SMD_Pin1Left
- moved SW1 231.8 mm to (167.8, 79.6)
- moved SW2 231.8 mm to (167.8, 67.5)
- moved SW3 231.8 mm to (167.8, 55.2)
- moved SW5 208.4 mm to (168.7, 91.0), turned to 180 degrees
- moved R14 204.5 mm to (164.9, 90.9), turned to 90 degrees
- moved J47 190.6 mm to (143.4, 37.3)
- moved C61 186.3 mm to (149.8, 49.2)
- moved C19 186.3 mm to (145.3, 48.5), turned to 180 degrees
- moved R59 184.3 mm to (143.7, 46.9), turned to 180 degrees
- moved R84 182.0 mm to (130.8, 130.6)
- moved R24 182.0 mm to (132.3, 131.7)
- moved R60 181.3 mm to (141.1, 45.3)
- moved R58 181.0 mm to (140.7, 47.7), turned to -90 degrees
- moved J74 180.4 mm to (133.4, 143.8)
- moved C60 180.3 mm to (146.2, 53.5), turned to -90 degrees
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- renumbered J3 to J1
Connections:
- net /5V renamed 5V
- net /chewing-gums/GPIO_17 renamed /GPIO_17
- net /chewing-gums/GPIO_18 renamed /GPIO_18
- net /chewing-gums/GPIO_19 renamed /GPIO_19
- net /chewing-gums/GPIO_20 renamed /GPIO_20
- net /chewing-gums/GPIO_21 renamed /GPIO_21
- net /chewing-gums/GPIO_22 renamed /GPIO_22
- net /chewing-gums/GPIO_24 renamed /GPIO_24
- net /chewing-gums/GPIO_25 renamed /GPIO_25
- net /chewing-gums/Vout_10_A renamed /Vout_A_10
- net /chewing-gums/Vout_11_A renamed /Vout_A_11
- net /chewing-gums/Vout_12_A renamed /Vout_A_12
- net /chewing-gums/Vout_1_A renamed /Vout_A_1
- net /chewing-gums/Vout_1_B renamed /Vout_B_0
- net /chewing-gums/Vout_1_diff renamed /Vout_diff_0
- net /chewing-gums/Vout_4_A renamed /Vout_A_4
- net /chewing-gums/Vout_4_diff renamed /Vout_diff_3
- net /chewing-gums/Vout_5_diff renamed /Vout_diff_4
- net /chewing-gums/Vout_6_diff renamed /Vout_diff_5
- net /chewing-gums/Vout_7_A renamed /Vout_A_7
- net /chewing-gums/Vout_8_A renamed /Vout_A_8
- net /chewing-gums/Vout_9_A renamed /Vout_A_9
- C16 pad 1: /VDD_IO -> VDD_IO_main
- C35 pad 1: /VDD_IO -> VDD_IO_main
- C36 pad 1: /VDD_IO -> VDD_IO_main
- C37 pad 1: /VDD_IO -> VDD_IO_main
- C38 pad 1: /VDD_IO -> VDD_IO_main
- C49 pad 1: /VDD_IO -> VDD_IO_main
- C85 pad 1: /VDD_IO -> VDD_IO_main
- C86 pad 1: /VDD_IO -> VDD_IO_main
- C90 pad 1: /VDD_IO -> VDD_IO_main
- CG1 pad 11: /chewing-gums/EN_1 -> /EN_CG_1
- CG1 pad 15: /A3V3 -> /A3V3_A
- CG1 pad 16: /REF -> /REF_A
- CG10 pad 11: /chewing-gums/EN_10 -> /EN_CG_10
- CG10 pad 15: /A3V3 -> /A3V3_B
- CG10 pad 16: /REF -> /REF_B
- CG10 pad 19: /chewing-gums/Vout_10_B -> /Vout_B_9
- CG10 pad 20: /chewing-gums/Vout_10_diff -> /Vout_diff_9
- CG11 pad 11: /chewing-gums/EN_11 -> /EN_CG_11
- CG11 pad 15: /A3V3 -> /A3V3_B
- CG11 pad 16: /REF -> /REF_B
- CG11 pad 19: /chewing-gums/Vout_11_B -> /Vout_B_10
- CG11 pad 20: /chewing-gums/Vout_11_diff -> /Vout_diff_10
- CG12 pad 11: /chewing-gums/EN_12 -> /EN_CG_12
- CG12 pad 15: /A3V3 -> /A3V3_B
- CG12 pad 16: /REF -> /REF_B
- CG12 pad 19: /chewing-gums/Vout_12_B -> /Vout_B_11
- CG12 pad 20: /chewing-gums/Vout_12_diff -> /Vout_diff_11
- CG2 pad 1: /chewing-gums/Vout_2_A -> /Vout_A_2
- CG2 pad 11: /chewing-gums/EN_2 -> /EN_CG_2
- CG2 pad 15: /A3V3 -> /A3V3_A
- CG2 pad 16: /REF -> /REF_A
- CG2 pad 19: /chewing-gums/Vout_2_B -> /Vout_B_1
- CG2 pad 2: /chewing-gums/Vout_2_A -> /Vout_A_2
- CG2 pad 20: /chewing-gums/Vout_2_diff -> /Vout_diff_1
- CG2 pad 21: /chewing-gums/Vout_2_A -> /Vout_A_2
- CG3 pad 1: /chewing-gums/Vout_3_A -> /Vout_A_3
- CG3 pad 11: /chewing-gums/EN_3 -> /EN_CG_3
- CG3 pad 15: /A3V3 -> /A3V3_A
- CG3 pad 16: /REF -> /REF_A
- CG3 pad 19: /chewing-gums/Vout_3_B -> /Vout_B_2
- CG3 pad 2: /chewing-gums/Vout_3_A -> /Vout_A_3
- CG3 pad 20: /chewing-gums/Vout_3_diff -> /Vout_diff_2
- CG3 pad 21: /chewing-gums/Vout_3_A -> /Vout_A_3
- CG4 pad 11: /chewing-gums/EN_4 -> /EN_CG_4
- CG4 pad 15: /A3V3 -> /A3V3_A
- CG4 pad 16: /REF -> /REF_A
- CG4 pad 19: /chewing-gums/Vout_4_B -> /Vout_B_3
- CG5 pad 1: /VDD_IO -> VDD_IO_cheep
- CG5 pad 11: /chewing-gums/EN_5 -> /EN_CG_5
- CG5 pad 15: /A3V3 -> /A3V3_A
- CG5 pad 16: /REF -> /REF_A
- CG5 pad 19: /chewing-gums/Vout_5_B -> /Vout_B_4
- CG5 pad 2: /VDD_IO -> VDD_IO_cheep
- CG5 pad 21: /VDD_IO -> VDD_IO_cheep
- CG6 pad 1: /chewing-gums/Vout_6_A -> VDD_IO_main
- CG6 pad 11: /chewing-gums/EN_6 -> /EN_CG_6
- CG6 pad 15: /A3V3 -> /A3V3_A
- CG6 pad 16: /REF -> /REF_A
- CG6 pad 19: /chewing-gums/Vout_6_B -> /Vout_B_5
- CG6 pad 2: /chewing-gums/Vout_6_A -> VDD_IO_main
- CG6 pad 21: /chewing-gums/Vout_6_A -> VDD_IO_main
- CG7 pad 11: /chewing-gums/EN_7 -> /EN_CG_7
- CG7 pad 15: /A3V3 -> /A3V3_B
- CG7 pad 16: /REF -> /REF_B
- CG7 pad 19: /chewing-gums/Vout_7_B -> /Vout_B_6
- CG7 pad 20: /chewing-gums/Vout_7_diff -> /Vout_diff_6
- CG8 pad 11: /chewing-gums/EN_8 -> /EN_CG_8
- CG8 pad 15: /A3V3 -> /A3V3_B
- CG8 pad 16: /REF -> /REF_B
- CG8 pad 19: /chewing-gums/Vout_8_B -> /Vout_B_7
- CG8 pad 20: /chewing-gums/Vout_8_diff -> /Vout_diff_7
- CG9 pad 11: /chewing-gums/EN_9 -> /EN_CG_9
- CG9 pad 15: /A3V3 -> /A3V3_B
- CG9 pad 16: /REF -> /REF_B
- CG9 pad 19: /chewing-gums/Vout_9_B -> /Vout_B_8
- CG9 pad 20: /chewing-gums/Vout_9_diff -> /Vout_diff_8
- IC10 pad 13: /VDD_IO -> VDD_IO_main
- IC15 pad 13: /VDD_IO -> VDD_IO_main
- IC16 pad 13: /VDD_IO -> VDD_IO_main
- IC2 pad 13: /VDD_IO -> VDD_IO_main
- IC3 pad 1: /EP_TRST -> /TX0
- IC3 pad 10: /RX0_LT -> /TRST_LT
- IC3 pad 11: /GPIO22 -> /RX0_LT
- IC3 pad 12: /TRST_LT -> /TX0_LT
- IC3 pad 13: /VDD_IO -> VDD_IO_main
- IC3 pad 2: /EP_A5 -> /RX0
- IC3 pad 3: /RX0 -> /EP_TRST
- IC3 pad 4: /TX0 -> /EP_A5
- IC3 pad 9: /TX0_LT -> /GPIO22
- IC4 pad 13: /VDD_IO -> VDD_IO_main
- J1 pad 10: /chewing-gums/GPIO_11 -> /GPIO_11
- J1 pad 11: /chewing-gums/GPIO_12 -> /GPIO_12
- J1 pad 12: /chewing-gums/GPIO_13 -> /GPIO_13
- J1 pad 13: /chewing-gums/GPIO_14 -> /GPIO_14
- J1 pad 14: /chewing-gums/GPIO_15 -> /GPIO_15
- J1 pad 15: /chewing-gums/GPIO_16 -> /GPIO_16
- J1 pad 29: unconnected-(J3-Pin_29-Pad29) -> /CHEEP-CONNECTOR/REF_A
- J1 pad 3: /chewing-gums/Vout_3_diff -> /Vout_B_1
- J1 pad 30: unconnected-(J3-Pin_30-Pad30) -> /CHEEP-CONNECTOR/REF_A
- J1 pad 31: unconnected-(J3-Pin_31-Pad31) -> /CHEEP-CONNECTOR/A3V3_A
- J1 pad 32: unconnected-(J3-Pin_32-Pad32) -> /CHEEP-CONNECTOR/A3V3_A
- J1 pad 4: /chewing-gums/Vout_3_B -> /Vout_diff_1
- J1 pad 5: /chewing-gums/Vout_3_A -> /Vout_A_2
- J1 pad 6: /chewing-gums/Vout_3_A -> /Vout_A_2
- J1 pad 9: /chewing-gums/GPIO_10 -> /GPIO_10
- R14 pad 2: /VDD_IO -> VDD_IO_main
- R27 pad 1: /VDD_IO -> VDD_IO_main
- R6 pad 1: /VDD_IO -> VDD_IO_main
- R7 pad 1: /VDD_IO -> VDD_IO_main
- R8 pad 1: /VDD_IO -> VDD_IO_main
- R9 pad 1: /VDD_IO -> VDD_IO_main
- SW1 pad 1: /VDD_IO -> VDD_IO_main
- SW2 pad 1: /VDD_IO -> VDD_IO_main
- SW3 pad 1: /VDD_IO -> VDD_IO_main
- U11 pad 2: /spi_flash_sd_1 -> /CHEEP-CONNECTOR/SPI_FLASH.SD1
- U11 pad 4: /spi_flash_Bs -> /CHEEP-CONNECTOR/SPI_FLASH.CS0
- U12 pad 2: /spi_flash_sck -> /CHEEP-CONNECTOR/SPI_FLASH.SCK
- U12 pad 4: /spi_flash_sd_2 -> /CHEEP-CONNECTOR/SPI_FLASH.SD2
- U13 pad 2: /spi_flash_sd_0 -> /CHEEP-CONNECTOR/SPI_FLASH.SD0
- U13 pad 4: /spi_flash_sd_3 -> /CHEEP-CONNECTOR/SPI_FLASH.SD3
- U2 pad 8: /VDD_IO -> VDD_IO_main
- U27 pad 7: /VDD_IO -> VDD_IO_main
- U4 pad 19: /chewing-gums/Vout_3_diff -> /Vout_diff_2
- U4 pad 23: /chewing-gums/Vout_10_diff -> unconnected-(U4-IO11-Pad23)
- U4 pad 24: /chewing-gums/Vout_9_diff -> unconnected-(U4-IO12-Pad24)
- U4 pad 25: /chewing-gums/Vout_8_diff -> unconnected-(U4-IO13-Pad25)
- U4 pad 26: /chewing-gums/Vout_7_diff -> unconnected-(U4-IO14-Pad26)
- U4 pad 29: /chewing-gums/DAC_4 -> unconnected-(U4-IO17-Pad29)
- U4 pad 30: /chewing-gums/DAC_5 -> unconnected-(U4-IO18-Pad30)
- U4 pad 31: /chewing-gums/DAC_6 -> unconnected-(U4-IO19-Pad31)
- U4 pad 32: /chewing-gums/DAC_7 -> unconnected-(U4-IO20-Pad32)
- U4 pad 37: /A3V3 -> /A3V3_A
- U4 pad 38: /A3V3 -> /A3V3_A
- U4 pad 39: /REF -> /REF_A
- U4 pad 40: /REF -> /REF_A
- X2 pad 4: /VDD_IO -> VDD_IO_main
Routing:
- net (no net): track 52.0 -> 423.9 mm
- net /SDA: track 349.5 -> 26.3 mm, vias 3 -> 2
- net GND: track 112.4 -> 336.6 mm, vias 18 -> 11
- net /REF: track 208.2 -> 0.00 mm
- net /A3V3: track 173.7 -> 0.00 mm
- net /SCL: track 190.4 -> 29.3 mm, vias 3 -> 2
- net 5V: track 219.2 -> 376.5 mm
- net unconnected-(U4-IO14-Pad26): track 0.00 -> 128.1 mm
- net /A3V3_A: track 0.00 -> 109.8 mm
- net /Vout_A_7: track 12.3 -> 120.5 mm
- net VDD_IO_main: track 0.00 -> 107.0 mm, vias 0 -> 2
- net VDD_IO_cheep: track 0.00 -> 104.5 mm
- net /VDD_IO: track 103.5 -> 0.00 mm, vias 4 -> 0
- net /REF_A: track 0.00 -> 103.1 mm
- net unconnected-(U4-IO11-Pad23): track 0.00 -> 100.1 mm
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- added copper zone on F.Cu, net /Programmer/VCORE
- added copper zone on F.Cu, net /VEXT
- added copper zone on In2.Cu, net 3V3
- added copper zone on In2.Cu, net 5V
- added copper zone on In1.Cu, net GND
- removed copper zone on B.Cu, net 3V3
- removed copper zone on B.Cu, net 5V
Other:
- board size 170.8 x 120.2 mm -> 143.6 x 128.4 mm
- board text added: "Change these for smaller vertical switches"
- board text added: "LVL shf"
- board text added: "NOT CONNECTED"
- board text added: "VDD IO cheep"
- board text added: "VDD IO main"

Commit message: WIP: added i2c expanders and re-structuring i2c distributino
Parts:
- removed C63, C64, C81, C85, C86: 0.1u, Capacitor_SMD:C_0603_1608Metric
- removed C82, C83: 100n, Capacitor_SMD:C_0603_1608Metric
- removed IC15, IC16: SN74AXC4T774RSVR, heep_footprints:TI-UQFN-16
- removed R101, R102, R70, R71, R72, R73, R74, R75: 100, Resistor_SMD:R_0603_1608Metric
- removed R103, R104, R105, R106, R107, R108, R109, R110, R111, R78: 10k, Resistor_SMD:R_0603_1608Metric
- removed SW1, SW2, SW3: SW_SPDT, Button_Switch_SMD:SW_SPDT_PCM12
- removed U24: TCA9554ADBQR, Package_SO:SSOP-16_3.9x4.9mm_P0.635mm
- added C18: 0.1u, Capacitor_SMD:C_0603_1608Metric, F.Cu at (177.9, 84.0)
- added C28: 100n, Capacitor_SMD:C_0603_1608Metric, F.Cu at (188.0, 129.7)
- added D1: LED, LED_SMD:LED_0603_1608Metric, F.Cu at (183.3, 115.2)
- added D2: LED, LED_SMD:LED_0603_1608Metric, F.Cu at (185.1, 115.2)
- added D3: LED, LED_SMD:LED_0603_1608Metric, F.Cu at (186.8, 115.2)
- added D4: LED, LED_SMD:LED_0603_1608Metric, F.Cu at (191.1, 115.1)
- added D5: LED, LED_SMD:LED_0603_1608Metric, F.Cu at (192.8, 115.1)
- added D6: LED, LED_SMD:LED_0603_1608Metric, F.Cu at (196.3, 115.2)
- added D8: LED, LED_SMD:LED_0603_1608Metric, F.Cu at (197.9, 115.2)
- added D9: LED, LED_SMD:LED_0603_1608Metric, F.Cu at (199.6, 115.2)
- added J8: Conn_01x03, Connector_PinHeader_2.54mm:PinHeader_1x03_P2.54mm_Vertical_SMD_Pin1Right, F.Cu at (175.9, 129.0)
- added R10: 1k, Resistor_SMD:R_0603_1608Metric, F.Cu at (146.1, 130.5)
- added R11: 1k, Resistor_SMD:R_0603_1608Metric, F.Cu at (146.3, 125.0)
- added R16: 1k, Resistor_SMD:R_0603_1608Metric, F.Cu at (146.2, 119.4)
- added R17: 1k, Resistor_SMD:R_0603_1608Metric, F.Cu at (183.3, 118.2)
- added R18: 1k, Resistor_SMD:R_0603_1608Metric, F.Cu at (185.0, 118.2)
- added R19: 1k, Resistor_SMD:R_0603_1608Metric, F.Cu at (186.8, 118.2)
- added R20: 1k, Resistor_SMD:R_0603_1608Metric, F.Cu at (191.1, 118.2)
- added R21: 1k, Resistor_SMD:R_0603_1608Metric, F.Cu at (192.8, 118.2)
- added R22: 1k, Resistor_SMD:R_0603_1608Metric, F.Cu at (196.3, 118.2)
- added R23: 1k, Resistor_SMD:R_0603_1608Metric, F.Cu at (197.9, 118.2)
- added R27: 1k, Resistor_SMD:R_0603_1608Metric, F.Cu at (199.6, 118.2)
- added SW4: SW_Push, Button_Switch_SMD:SW_Push_1P1T_NO_CK_KMR2, F.Cu at (144.9, 127.8)
- added SW6: SW_Push, Button_Switch_SMD:SW_Push_1P1T_NO_CK_KMR2, F.Cu at (145.0, 122.4)
- added SW7: SW_Push, Button_Switch_SMD:SW_Push_1P1T_NO_CK_KMR2, F.Cu at (144.9, 116.7)
- added U15: ~, heep_footprints:BIWIN_DTS04GE_SMD, F.Cu at (186.1, 99.8)
- added U16: ~, heep_footprints:BIWIN_DTS04GE_SMD, F.Cu at (149.6, 134.2)
- added U17: 74AHC244, Package_SO:TSSOP-20_4.4x6.5mm_P0.65mm, F.Cu at (191.0, 124.6)
- added U18: 74AHCT1G08, Package_TO_SOT_SMD:SOT-23-5, F.Cu at (198.5, 129.9)
- added U19: 74AHCT1G08, Package_TO_SOT_SMD:SOT-23-5, F.Cu at (198.4, 122.5)
- added U20: 74AHC1G04, Package_TO_SOT_SMD:SOT-23-5, F.Cu at (198.5, 126.1)
- added U21: TCA9548ARGER, Package_DFN_QFN:Texas_RGE0024C_VQFN-24-1EP_4x4mm_P0.5mm_EP2.1x2.1mm, F.Cu at (157.0, 100.7)
- added U22: TCA9548ARGER, Package_DFN_QFN:Texas_RGE0024C_VQFN-24-1EP_4x4mm_P0.5mm_EP2.1x2.1mm, F.Cu at (193.0, 101.0)
- added U8: TS5A23159DGS, heep_footprints:VSSOP-10_3x3mm_P0.5mm_sch, F.Cu at (178.1, 86.6)
- J6: renamed from J37; footprint Connector_PinSocket_2.54mm:PinSocket_1x03_P2.54mm_Vertical_SMD_Pin1Left -> Connector_PinHeader_2.54mm:PinHeader_1x03_P2.54mm_Vertical_SMD_Pin1Right
- R12, R13: value 100 -> 10k
- U11, U12, U13, U14, U28: footprint Package_SO:VSSOP-10_3x3mm_P0.5mm -> heep_footprints:VSSOP-10_3x3mm_P0.5mm_sch
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- renumbered C87 to C23, C49 to C24, C88 to C25, C89 to C26, C90 to C27, J74 to J7, R27 to R1, R82 to R4, R83 to R5, U27 to U10, X2 to X1
Connections:
- net /EP_F_BS renamed /EP_F_CS
- net /HEEP_BLOCK_SEL renamed /EP_CLOCK_SEL
- CG1 pad 19: /Vout_B_0 -> /Vout_B_1
- CG1 pad 20: /Vout_diff_0 -> /Vout_diff_1
- CG1 pad 6: /SCL -> /CG_I2C_SCL_1
- CG1 pad 7: /SDA -> /CG_I2C_SDA_1
- CG10 pad 19: /Vout_B_9 -> /Vout_B_10
- CG10 pad 20: /Vout_diff_9 -> /Vout_diff_10
- CG10 pad 6: /SCL -> /CG_I2C_SCL_10
- CG10 pad 7: /SDA -> /CG_I2C_SDA_10
- CG11 pad 19: /Vout_B_10 -> /Vout_B_11
- CG11 pad 20: /Vout_diff_10 -> /Vout_diff_11
- CG11 pad 6: /SCL -> /CG_I2C_SCL_11
- CG11 pad 7: /SDA -> /CG_I2C_SDA_11
- CG12 pad 19: /Vout_B_11 -> /Vout_B_12
- CG12 pad 20: /Vout_diff_11 -> /Vout_diff_12
- CG12 pad 6: /SCL -> /CG_I2C_SCL_12
- CG12 pad 7: /SDA -> /CG_I2C_SDA_12
- CG2 pad 19: /Vout_B_1 -> /Vout_B_2
- CG2 pad 20: /Vout_diff_1 -> /Vout_diff_2
- CG2 pad 6: /SCL -> /CG_I2C_SCL_2
- CG2 pad 7: /SDA -> /CG_I2C_SDA_2
- CG3 pad 19: /Vout_B_2 -> /Vout_B_3
- CG3 pad 20: /Vout_diff_2 -> /Vout_diff_3
- CG3 pad 6: /SCL -> /CG_I2C_SCL_3
- CG3 pad 7: /SDA -> /CG_I2C_SDA_3
- CG4 pad 19: /Vout_B_3 -> /Vout_B_4
- CG4 pad 20: /Vout_diff_3 -> /Vout_diff_4
- CG4 pad 6: /SCL -> /CG_I2C_SCL_4
- CG4 pad 7: /SDA -> /CG_I2C_SDA_4
- CG5 pad 19: /Vout_B_4 -> /Vout_B_5
- CG5 pad 20: /Vout_diff_4 -> /Vout_diff_5
- CG5 pad 6: /SCL -> /CG_I2C_SCL_5
- CG5 pad 7: /SDA -> /CG_I2C_SDA_5
- CG6 pad 19: /Vout_B_5 -> /Vout_B_6
- CG6 pad 20: /Vout_diff_5 -> /Vout_diff_6
- CG6 pad 6: /SCL -> /CG_I2C_SCL_6
- CG6 pad 7: /SDA -> /CG_I2C_SDA_6
- CG7 pad 19: /Vout_B_6 -> /Vout_B_7
- CG7 pad 20: /Vout_diff_6 -> /Vout_diff_7
- CG7 pad 6: /SCL -> /CG_I2C_SCL_7
- CG7 pad 7: /SDA -> /CG_I2C_SDA_7
- CG8 pad 19: /Vout_B_7 -> /Vout_B_8
- CG8 pad 20: /Vout_diff_7 -> /Vout_diff_8
- CG8 pad 6: /SCL -> /CG_I2C_SCL_8
- CG8 pad 7: /SDA -> /CG_I2C_SDA_8
- CG9 pad 19: /Vout_B_8 -> /Vout_B_9
- CG9 pad 20: /Vout_diff_8 -> /Vout_diff_9
- CG9 pad 6: /SCL -> /CG_I2C_SCL_9
- CG9 pad 7: /SDA -> /CG_I2C_SDA_9
- IC10 pad 10: /LevelTransMeasCurrent/FTDI_GPIO_8_VIO -> unconnected-(IC10-B3-Pad10)
- IC10 pad 11: /LevelTransMeasCurrent/HEEP_BLOCK_SEL_VIO -> /CLOCK_SEL
- IC10 pad 3: /EP_A6 -> unconnected-(IC10-A3-Pad3)
- IC10 pad 4: /EP_A7 -> unconnected-(IC10-A4-Pad4)
- IC10 pad 6: /LevelTransMeasCurrent/DIR4 -> Net-(IC10-DIR4)
- IC10 pad 9: /LevelTransMeasCurrent/FTDI_GPIO_9_VIO -> unconnected-(IC10-B4-Pad9)
- IC2 pad 10: /TMS_LT -> /CHEEP-CONNECTOR/JTAG.TDO
- IC2 pad 11: /TDI_LT -> /CHEEP-CONNECTOR/JTAG.TDI
- IC2 pad 12: /TCK_LT -> /CHEEP-CONNECTOR/JTAG.TCK
- IC2 pad 3: /EP_TMS -> /EP_TDO
- IC2 pad 4: /EP_TDO -> /EP_TMS
- IC2 pad 9: /TDO_LT -> /CHEEP-CONNECTOR/JTAG.TMS
- IC3 pad 1: /TX0 -> /EP_TRST
- IC3 pad 10: /TRST_LT -> /CHEEP-CONNECTOR/UART.RX
- IC3 pad 11: /RX0_LT -> unconnected-(IC3-B2-Pad11)
- IC3 pad 12: /TX0_LT -> /CHEEP-CONNECTOR/JTAG.TRST
- IC3 pad 2: /RX0 -> unconnected-(IC3-A2-Pad2)
- IC3 pad 3: /EP_TRST -> /EP_RX0
- IC3 pad 4: /EP_A5 -> /EP_TX0
- IC3 pad 9: /GPIO22 -> /CHEEP-CONNECTOR/UART.TX
- IC4 pad 12: /LevelTransMeasCurrent/FLASH_BS_FTDI_VIO -> /LevelTransMeasCurrent/FLASH_CS_FTDI_VIO
- J1 pad 24: /GPIO_22 -> /GPIO_23
- J1 pad 29: /CHEEP-CONNECTOR/REF_A -> /REF_A
- J1 pad 3: /Vout_B_1 -> /Vout_B_2
- J1 pad 30: /CHEEP-CONNECTOR/REF_A -> /REF_A
- J1 pad 31: /CHEEP-CONNECTOR/A3V3_A -> /A3V3_A
- J1 pad 32: /CHEEP-CONNECTOR/A3V3_A -> /A3V3_A
- J1 pad 4: /Vout_diff_1 -> /Vout_diff_2
- J2 pad 1: /Vout_B_2 -> /Vout_B_3
- J2 pad 10: /CHEEP-CONNECTOR/EXIT_VALUE -> /EXIT_VALUE
- J2 pad 11: /CHEEP-CONNECTOR/BOOT_SEL -> /BOOT_SEL
- J2 pad 12: unconnected-(J2-Pin_12-Pad12) -> /EXEC_FLASH
- J2 pad 2: /Vout_diff_2 -> /Vout_diff_3
- J2 pad 7: /CHEEP-CONNECTOR/nRST -> /nRST
- J2 pad 8: /CHEEP-CONNECTOR/EXEC_FLASH -> unconnected-(J2-Pin_8-Pad8)
- J2 pad 9: /CHEEP-CONNECTOR/EXIT_VALID -> /EXIT_VALID
- J3 pad 1: /CHEEP-CONNECTOR/Vout_5_B -> /Vout_B_5
- J3 pad 15: /CHEEP-CONNECTOR/JTAG_TCK -> /CHEEP-CONNECTOR/JTAG.TCK
- J3 pad 16: /CHEEP-CONNECTOR/JTAG_TMS -> /CHEEP-CONNECTOR/JTAG.TMS
- J3 pad 17: /CHEEP-CONNECTOR/JTAG_TD0 -> /CHEEP-CONNECTOR/JTAG.TDO
- J3 pad 18: /CHEEP-CONNECTOR/JTAG_TDI -> /CHEEP-CONNECTOR/JTAG.TDI
- J3 pad 19: GND -> /CHEEP-CONNECTOR/JTAG.TRST
- J3 pad 2: /Vout_diff_4 -> /Vout_diff_5
- J3 pad 21: /CHEEP-CONNECTOR/UART_TX -> /CHEEP-CONNECTOR/UART.TX
- J3 pad 22: /CHEEP-CONNECTOR/UART_RX -> /CHEEP-CONNECTOR/UART.RX
- J3 pad 25: /Vout_B_3 -> /Vout_B_4
- J3 pad 26: /Vout_diff_3 -> /Vout_diff_4
- J3 pad 31: /CHEEP-CONNECTOR/clk -> /CLOCK
- J4 pad 13: /Vout_B_9 -> /Vout_B_10
- J4 pad 14: /Vout_diff_9 -> /Vout_diff_10
- J4 pad 17: /Vout_B_8 -> /Vout_B_9
- J4 pad 18: /Vout_diff_8 -> /Vout_diff_9
- J4 pad 23: /Vout_B_7 -> /Vout_B_8
- J4 pad 24: /Vout_diff_7 -> /Vout_diff_8
- J4 pad 27: /Vout_B_6 -> /Vout_B_7
- J4 pad 28: /Vout_diff_6 -> /Vout_diff_7
- J4 pad 3: /Vout_B_11 -> /Vout_B_12
- J4 pad 4: /Vout_diff_11 -> /Vout_diff_12
- J4 pad 7: /Vout_B_10 -> /Vout_B_11
- J4 pad 8: /Vout_diff_10 -> /Vout_diff_11
- J5 pad 1: /CHEEP-CONNECTOR/REF_B -> /REF_B
- J5 pad 10: /CHEEP-CONNECTOR/SCL -> /CHEEP-CONNECTOR/CHEEP_I2C.SCL
- J5 pad 2: /CHEEP-CONNECTOR/REF_B -> /REF_B
- J5 pad 5: /CHEEP-CONNECTOR/A3V3_B -> /A3V3_B
- J5 pad 6: /CHEEP-CONNECTOR/A3V3_B -> /A3V3_B
- J5 pad 9: /CHEEP-CONNECTOR/SDA -> /CHEEP-CONNECTOR/CHEEP_I2C.SDA
- J6 pad 1: /LevelTransMeasCurrent/HEEP_BLOCK_SEL_VIO -> GND
- J6 pad 3: GND -> /CLOCK_SEL
- J68 pad 2: /LevelTransMeasCurrent/DIR3 -> Net-(IC10-DIR4)
- J68 pad 4: /LevelTransMeasCurrent/DIR4 -> /LevelTransMeasCurrent/DIR3
- J7 pad 1: /CLK_HEEP -> /CLOCK
- J71 pad 2: Net-(IC2-~{OE}) -> GND
- J73 pad 2: /TX0_LT -> /CHEEP-CONNECTOR/UART.TX
- J73 pad 3: /RX0_LT -> /CHEEP-CONNECTOR/UART.RX
- R12 pad 1: /GPIO8 -> VDD_IO_main
- R12 pad 2: /LevelTransMeasCurrent/FTDI_GPIO_8_VIO -> /CHEEP-CONNECTOR/CHEEP_I2C.SDA
- R13 pad 1: /GPIO9 -> VDD_IO_main
- R13 pad 2: /LevelTransMeasCurrent/FTDI_GPIO_9_VIO -> /CHEEP-CONNECTOR/CHEEP_I2C.SCL
- R14 pad 1: /nRST_HEEP -> /nRST
- R24 pad 2: /SCL -> SCL
- R4 pad 1: /CLK_HEEP -> Net-(J8-Pin_3)
- R5 pad 1: /CLK_HEEP -> Net-(J8-Pin_1)
- R6 pad 2: /LevelTransMeasCurrent/FLASH_BS -> /LevelTransMeasCurrent/FLASH_CS
- R77 pad 1: /LevelTransMeasCurrent/DIR4 -> Net-(IC10-DIR4)
- R84 pad 2: /SDA -> SDA
- SW5 pad 1: /nRST_HEEP -> /nRST
- U1 pad 22: /EP_A5 -> unconnected-(U1-ADBUS5-Pad22)
- U1 pad 23: /EP_A6 -> unconnected-(U1-ADBUS6-Pad23)
- U1 pad 24: /EP_A7 -> unconnected-(U1-ADBUS7-Pad24)
- U1 pad 29: /Programmer/SPI_BS -> unconnected-(U1-BDBUS3-Pad29)
- U1 pad 38: /RX0 -> /EP_TX0
- U1 pad 39: /TX0 -> /EP_RX0
- U1 pad 40: /Programmer/C2 -> unconnected-(U1-CDBUS2-Pad40)
- U1 pad 41: /Programmer/C3 -> unconnected-(U1-CDBUS3-Pad41)
- U1 pad 43: /Programmer/C4 -> unconnected-(U1-CDBUS4-Pad43)
- U1 pad 44: /Programmer/C5 -> unconnected-(U1-CDBUS5-Pad44)
- U1 pad 45: /Programmer/C6 -> unconnected-(U1-CDBUS6-Pad45)
- U1 pad 46: /Programmer/C7 -> unconnected-(U1-CDBUS7-Pad46)
- U1 pad 48: /EP_D0 -> unconnected-(U1-DDBUS0-Pad48)
- U1 pad 52: /EP_D1 -> unconnected-(U1-DDBUS1-Pad52)
- U1 pad 53: /EP_D2 -> unconnected-(U1-DDBUS2-Pad53)
- U1 pad 54: /EP_D3 -> unconnected-(U1-DDBUS3-Pad54)
- U1 pad 55: /EP_D4 -> unconnected-(U1-DDBUS4-Pad55)
- U1 pad 57: /EP_D5 -> unconnected-(U1-DDBUS5-Pad57)
- U1 pad 58: /EP_D6 -> unconnected-(U1-DDBUS6-Pad58)
- U1 pad 59: /EP_D7 -> unconnected-(U1-DDBUS7-Pad59)
- U10 pad 4: /SCL -> SCL_LEFT
- U10 pad 5: /SDA -> SDA_LEFT
- U11 pad 10: /LevelTransMeasCurrent/FLASH_MISO -> /LevelTransMeasCurrent/FLASH_nWP
- U11 pad 2: /CHEEP-CONNECTOR/SPI_FLASH.SD1 -> /CHEEP-CONNECTOR/SPI_FLASH.SD2
- U11 pad 4: /CHEEP-CONNECTOR/SPI_FLASH.CS0 -> /CHEEP-CONNECTOR/SPI_FLASH.SD1
- U11 pad 6: /LevelTransMeasCurrent/FLASH_BS -> /LevelTransMeasCurrent/FLASH_MISO
- U11 pad 7: /LevelTransMeasCurrent/FLASH_BS_FTDI_VIO -> /LevelTransMeasCurrent/FLASH_MISO_FTDI_VIO
- U11 pad 9: /LevelTransMeasCurrent/FLASH_MISO_FTDI_VIO -> unconnected-(U11-Pad9)
- U12 pad 10: /LevelTransMeasCurrent/FLASH_SCK -> /LevelTransMeasCurrent/FLASH_CS
- U12 pad 2: /CHEEP-CONNECTOR/SPI_FLASH.SCK -> /CHEEP-CONNECTOR/SPI_FLASH.CS0
- U12 pad 4: /CHEEP-CONNECTOR/SPI_FLASH.SD2 -> /CHEEP-CONNECTOR/SPI_FLASH.SD3
- U12 pad 6: /LevelTransMeasCurrent/FLASH_nWP -> /LevelTransMeasCurrent/FLASH_nHLD_nRST
- U12 pad 9: /LevelTransMeasCurrent/FLASH_SCK_FTDI_VIO -> /LevelTransMeasCurrent/FLASH_CS_FTDI_VIO
- U13 pad 4: /CHEEP-CONNECTOR/SPI_FLASH.SD3 -> /CHEEP-CONNECTOR/SPI_FLASH.SCK
- U13 pad 6: /LevelTransMeasCurrent/FLASH_nHLD_nRST -> /LevelTransMeasCurrent/FLASH_SCK
- U13 pad 7: unconnected-(U13-Pad7) -> /LevelTransMeasCurrent/FLASH_SCK_FTDI_VIO
- U14 pad 1: /nRST_HEEP_FTDI -> unconnected-(U14-Pad1)
- U14 pad 10: Net-(IC10-B1) -> unconnected-(U14-Pad10)
- U14 pad 4: /SCL -> SCL
- U14 pad 9: /nRST_HEEP -> unconnected-(U14-Pad9)
- U2 pad 1: /LevelTransMeasCurrent/FLASH_BS -> /LevelTransMeasCurrent/FLASH_CS
- U28 pad 10: /Programmer/FLASH_MOSI_SDA -> /Programmer/FLASH_MISO_SDA
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Routing:
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- added copper zone on F.Cu, net (none)
- added copper zone on In2.Cu, net GND
Other:
- board text added: "Add ground at the end try to shield it Add the option of adding TH decaps to clean the power sources Add testpoints Add holes to add supports round edges"
- board text added: "BOOT"
- board text added: "CLK"
- board text added: "Change uUSB to USB C Add VDD IO main voltage regulator on main board Take VDD IO main to cheep connector on the rightmost connector"
- board text added: "Chewing gums ENABLE through I2C"
- board text added: "FLASH"
- board text added: "FTDI"
- board text added: "GPIOs"
- board text added: "GPIOs FTDI"
- board text added: "L/S"
- board text added: "L/S JTAG, UART"
- board text added: "LEDs"
- board text added: "LEVEL SHIFT (3V3/VIO)"
- board text added: "Master sel. for FLASH"
- board text added: "Master select for RST"
- board text added: "SPI flash FTDI"
- board text added: "SPI flash VIO"
- board text added: "SPI/I2C sel"
- board text added: "TRASH"
- board text removed: "Change these for smaller vertical switches"
- board text removed: "Clock"
- board text removed: "Fix the order here Add ground at the end try to shield it Add the option of adding TH decaps to clean the power sources"
- board text removed: "LVL shf"
- board text removed: "Programmer & LS"
