File: chewing-gums/1p6V_to_m1p6V_bias_gum/1p6V_to_m1p6V_bias_gum.kicad_sch (KiCad schematic)
At the start: 26 parts, among them J1 Conn_Coaxial, U1 LT1118, U2 TPS72301, U3 TLV75801PDBV, U4 MCP4726, U5 24AA02E-OT

Commit message: production files
Parts:
- removed R9: 10k, Resistor_SMD:R_0603_1608Metric, symbol Device:R_Small
- added R11: 10k, Resistor_SMD:R_0603_1608Metric, symbol Device:R_Small
- added TP1, TP2, TP4: 5029, TestPoint:TestPoint_Loop_D1.80mm_Drill1.0mm_Beaded, symbol dk_Test-Points:5029
- added TP3: 5029, TestPoint:TestPoint_Keystone_5019_Miniature, symbol dk_Test-Points:5029
- C1, C10, C2: LCSC C19702 -> C1590
- C3: LCSC C19702 -> C1607
- C4, C6, C7, C9: value 1u -> 10u
- C5: value 1u -> 2.2u; LCSC C19702 -> C1607
- R1: LCSC C98220 -> C25976
- R10: footprint Resistor_SMD:R_0603_1608Metric -> Resistor_SMD:R_0402_1005Metric; LCSC C98220 -> C25530
- R2: LCSC C98220 -> C23034
- R3, R5: value 33.2k -> 53.6k; LCSC C98220 -> C23074
- R4: value 7.03k -> 11.3k; LCSC C98220 -> C22860
- R6: value 1k -> 10k; now fitted
- R8: footprint Resistor_SMD:R_0603_1608Metric -> Resistor_SMD:R_0402_1005Metric; LCSC C98220 -> C25545
- U1: footprint heep-footprints:S8-package -> Package_SO:SOIC-8_3.9x4.9mm_P1.27mm
- U2: LCSC (none) -> C34678
- U4: footprint Package_TO_SOT_SMD:TSOT-23-6_HandSoldering -> Package_TO_SOT_SMD:TSOT-23-6; LCSC (none) -> C191581
- U5: LCSC (none) -> C38987
Connections:
- net -3.3VA: now also R11.1, TP2.1
- net -5V: no longer U2.3 (EN)
- net 3.3V: now also C2.1, U4.3 (VDD); no longer C2.2
- net 3.3VA: now also C1.1, C5.1, U4.6 (Vref), TP1.1; no longer U1.3 (EN)
- net GND: now also C2.2, U2.1 (GND), R11.2, TP3.1
- net V_bias: now also TP4.1
- net 5V: now reaches C9.1, U3.1 (IN)
- net 5V: now also CG1.A1 (5V), CG1.B1 (5V)
- net enable: now reaches CG1.B4 (ENABLE)
- net enable: now also U1.3 (EN), U2.3 (EN), U3.3 (EN)
- no-connect marks 5 -> 2
Other:
- note removed: "In case we need a load for stability"
